Commit message: break out gripper

File: fetch_description/robots/macros.xacro (robot description, xacro)
@@ -136,3 +136,80 @@
     </joint>
   </xacro:macro>
+  <xacro:macro name="gripper" params="base_link_name">
+  <link name="${base_link_name}">
+    <inertial>
+      <origin rpy="0 0 0" xyz="-0.0900 -0.0001 -0.0017" />
+      <mass value="1.5175" />
+      <inertia ixx="0.0013" ixy="-0.0" ixz="0.0" iyx="-0.0" iyy="0.0019" iyz="-0.0" izx="0.0" izy="-0.0" izz="0.0024" />
+    </inertial>
+    <visual>
+      <origin rpy="0 0 0" xyz="0 0 0" />
+      <geometry>
+        <mesh filename="package://fetch_description/meshes/gripper_link.dae" />
+      </geometry>
+    </visual>
+    <collision>
+      <origin rpy="0 0 0" xyz="0 0 0" />
+      <geometry>
+        <mesh filename="package://fetch_description/meshes/gripper_link.STL" />
+      </geometry>
+    </collision>
+  </link>
+    <link name="r_gripper_finger_link">
+      <inertial>
+        <origin rpy="0 0 0" xyz="-0.01 0 0" />
+        <mass value="0.0798" />
+        <inertia ixx="0.002" ixy="0" ixz="0" iyx="0.002" iyy="0" iyz="0" izx="0.002" izy="0" izz="0" />
+      </inertial>
+      <visual>
+        <origin rpy="0 0 0" xyz="0 0.101425 0" />
+        <geometry>
+          <mesh filename="package://fetch_description/meshes/r_gripper_finger_link.STL" />
+        </geometry>
+        <material name="">
+          <color rgba="0.356 0.361 0.376 1" />
+        </material>
+      </visual>
+      <collision>
+        <origin rpy="0 0 0" xyz="0 0.101425 0" />
+        <geometry>
+          <mesh filename="package://fetch_description/meshes/r_gripper_finger_link.STL" />
+        </geometry>
+      </collision>
+    </link>
+    <joint name="r_gripper_finger_joint" type="prismatic">
+      <origin rpy="0 0 0" xyz="0 0.015425 0" />
+      <parent link="${base_link_name}" />
+      <child link="r_gripper_finger_link" />
+      <axis xyz="0 1 0" />
+    <limit effort="60" lower="0.0" upper="0.05" velocity="0.05" /><dynamics damping="100.0" /></joint>
+    <link name="l_gripper_finger_link">
+      <inertial>
+        <origin rpy="0 0 0" xyz="-0.01 0 0" />
+        <mass value="0.0798" />
+        <inertia ixx="0.002" ixy="0" ixz="0" iyx="0.002" iyy="0" iyz="0" izx="0.002" izy="0" izz="0" />
+      </inertial>
+      <visual>
+        <origin rpy="0 0 0" xyz="0 -0.101425 0" />
+        <geometry>
+          <mesh filename="package://fetch_description/meshes/l_gripper_finger_link.STL" />
+        </geometry>
+        <material name="">
+          <color rgba="0.356 0.361 0.376 1" />
+        </material>
+      </visual>
+      <collision>
+        <origin rpy="0 0 0" xyz="0 -0.101425 0" />
+        <geometry>
+          <mesh filename="package://fetch_description/meshes/l_gripper_finger_link.STL" />
+        </geometry>
+      </collision>
+    </link>
+    <joint name="l_gripper_finger_joint" type="prismatic">
+      <origin rpy="0 0 0" xyz="0 -0.015425 0" />
+      <parent link="${base_link_name}" />
+      <child link="l_gripper_finger_link" />
+      <axis xyz="0 -1 0" />
+    <limit effort="60" lower="0.0" upper="0.05" velocity="0.05" /><dynamics damping="100.0" /></joint>
+  </xacro:macro>
 </robot>
