Commit message: Gripper abstracted out

File: fetch_description/robots/fetch.urdf.xacro (robot description, xacro)
@@ -2,479 +2,5 @@
   <xacro:include filename="$(find fetch_description)/robots/macros.xacro"/>
   <xacro:freight_macro velocity_limit="17.4" />
-  <link name="torso_lift_link">
-    <inertial>
-      <origin rpy="0 0 0" xyz="-0.0013 -0.0009 0.2935" />
-      <mass value="10.7796" />
-      <inertia ixx="0.3354" ixy="0.0" ixz="-0.0162" iyx="0.0" iyy="0.3354" iyz="-0.0006" izx="-0.0162" izy="-0.0006" izz="0.0954" />
-    </inertial>
-    <visual>
-      <origin rpy="0 0 0" xyz="0 0 0" />
-      <geometry>
-        <mesh filename="package://fetch_description/meshes/torso_lift_link.dae" />
-      </geometry>
-      <material name="">
-        <color rgba="1 1 1 1" />
-      </material>
-    </visual>
-    <collision>
-      <origin rpy="0 0 0" xyz="0 0 0" />
-      <geometry>
-        <mesh filename="package://fetch_description/meshes/torso_lift_link_collision.STL" />
-      </geometry>
-    </collision>
-  </link>
-  <joint name="torso_lift_joint" type="prismatic">
-    <origin rpy="-6.123E-17 0 0" xyz="-0.086875 0 0.37743" />
-    <parent link="base_link" />
-    <child link="torso_lift_link" />
-    <axis xyz="0 0 1" />
-    <limit effort="450.0" lower="0" upper="0.4" velocity="0.1" />
-  <dynamics damping="100.0" /></joint>
-  <link name="head_pan_link">
-    <inertial>
-      <origin rpy="0 0 0" xyz="0.0321 0.0161 0.0390" />
-      <mass value="2.2556" />
-      <inertia ixx="0.0129" ixy="0.0002" ixz="0.0007" iyx="0.0002" iyy="0.0095" iyz="-0.0" izx="0.0007" izy="-0.0" izz="0.0184" />
-    </inertial>
-    <visual>
-      <origin rpy="0 0 0" xyz="0 0 0" />
-      <geometry>
-        <mesh filename="package://fetch_description/meshes/head_pan_link.dae" />
-      </geometry>
-      <material name="">
-        <color rgba="0.356 0.361 0.376 1" />
-      </material>
-    </visual>
-    <collision>
-      <origin rpy="0 0 0" xyz="0 0 0" />
-      <geometry>
-        <mesh filename="package://fetch_description/meshes/head_pan_link_collision.STL" />
-      </geometry>
-    </collision>
-  </link>
-  <joint name="head_pan_joint" type="revolute">
-    <origin rpy="0 0 0" xyz="0.053125 0 0.603001417713939" />
-    <parent link="torso_lift_link" />
-    <child link="head_pan_link" />
-    <axis xyz="0 0 1" />
-  <limit effort="0.32" lower="-1.57" upper="1.57" velocity="1.57" /></joint>
-  <link name="head_tilt_link">
-    <inertial>
-      <origin rpy="0 0 0" xyz="0.0081 0.0025 0.0113" />
-      <mass value="0.9087" />
-      <inertia ixx="0.0061" ixy="-0.0" ixz="0.0002" iyx="-0.0" iyy="0.0014" iyz="-0.0001" izx="0.0002" izy="-0.0001" izz="0.0061" />
-    </inertial>
-    <visual>
-      <origin rpy="0 0 0" xyz="0 0 0" />
-      <geometry>
-        <mesh filename="package://fetch_description/meshes/head_tilt_link.dae" />
-      </geometry>
-      <material name="">
-        <color rgba="0.086 0.506 0.767 1" />
-      </material>
-    </visual>
-    <collision>
-      <origin rpy="0 0 0" xyz="0 0 0" />
-      <geometry>
-        <mesh filename="package://fetch_description/meshes/head_tilt_link_collision.STL" />
-      </geometry>
-    </collision>
-  </link>
-  <joint name="head_tilt_joint" type="revolute">
-    <origin rpy="0 0 0" xyz="0.14253 0 0.057999" />
-    <parent link="head_pan_link" />
-    <child link="head_tilt_link" />
-    <axis xyz="0 1 0" />
-    <limit effort="0.68" lower="-0.76" upper="1.45" velocity="1.57" />
-  </joint>
-  <link name="shoulder_pan_link">
-    <inertial>
-      <origin rpy="0 0 0" xyz="0.0927 -0.0056 0.0564" />
-      <mass value="2.5587" />
-      <inertia ixx="0.0043" ixy="-0.0001" ixz="0.001" iyx="-0.0001" iyy="0.0087" iyz="-0.0001" izx="0.001" izy="-0.0001" izz="0.0087" />
-    </inertial>
-    <visual>
-      <origin rpy="0 0 0" xyz="0 0 0" />
-      <geometry>
-        <mesh filename="package://fetch_description/meshes/shoulder_pan_link.dae" />
-      </geometry>
-      <material name="">
-        <color rgba="1 1 1 1" />
-      </material>
-    </visual>
-    <collision>
-      <origin rpy="0 0 0" xyz="0 0 0" />
-      <geometry>
-        <mesh filename="package://fetch_description/meshes/shoulder_pan_link_collision.STL" />
-      </geometry>
-    </collision>
-  </link>
-  <joint name="shoulder_pan_joint" type="revolute">
-    <origin rpy="0 0 0" xyz="0.119525 0 0.34858" />
-    <parent link="torso_lift_link" />
-    <child link="shoulder_pan_link" />
-    <axis xyz="0 0 1" />
-  <limit effort="33.82" lower="-1.6056" upper="1.6056" velocity="1.256" /></joint>
-  <link name="shoulder_lift_link">
-    <inertial>
-      <origin rpy="0 0 0" xyz="0.1432 0.0072 -0.0001" />
-      <mass value="2.6615" />
-      <inertia ixx="0.0028" ixy="-0.0021" ixz="-0.0" iyx="-0.0021" iyy="0.0111" iyz="-0.0" izx="-0.0" izy="-0.0" izz="0.0112" />
-    </inertial>
-    <visual>
-      <origin rpy="0 0 0" xyz="0 0 0" />
-      <geometry>
-        <mesh filename="package://fetch_description/meshes/shoulder_lift_link.dae" />
-      </geometry>
-      <material name="">
-        <color rgba="0.086 0.506 0.767 1" />
-      </material>
-    </visual>
-    <collision>
-      <origin rpy="0 0 0" xyz="0 0 0" />
-      <geometry>
-        <mesh filename="package://fetch_description/meshes/shoulder_lift_link_collision.STL" />
-      </geometry>
-    </collision>
-  </link>
-  <joint name="shoulder_lift_joint" type="revolute">
-    <origin rpy="0 0 0" xyz="0.117 0 0.0599999999999999" />
-    <parent link="shoulder_pan_link" />
-    <child link="shoulder_lift_link" />
-    <axis xyz="0 1 0" />
-  <limit effort="131.76" lower="-1.221" upper="1.518" velocity="1.454" /></joint>
-  <link name="upperarm_roll_link">
-    <inertial>
-      <origin rpy="0 0 0" xyz="0.1165 0.0014 0.0000" />
-      <mass value="2.3311" />
-      <inertia ixx="0.0019" ixy="-0.0001" ixz="0.0" iyx="-0.0001" iyy="0.0045" iyz="0.0" izx="0.0" izy="0.0" izz="0.0047" />
-    </inertial>
-    <visual>
-      <origin rpy="0 0 0" xyz="0 0 0" />
-      <geometry>
-        <mesh filename="package://fetch_description/meshes/upperarm_roll_link.dae" />
-      </geometry>
-      <material name="">
-        <color rgba="1 1 1 1" />
-      </material>
-    </visual>
-    <collision>
-      <origin rpy="0 0 0" xyz="0 0 0" />
-      <geometry>
-        <mesh filename="package://fetch_description/meshes/upperarm_roll_link_collision.STL" />
-      </geometry>
-    </collision>
-  </link>
-  <joint name="upperarm_roll_joint" type="continuous">
-    <origin rpy="0 0 0" xyz="0.219 0 0" />
-    <parent link="shoulder_lift_link" />
-    <child link="upperarm_roll_link" />
-    <axis xyz="1 0 0" />
-  <limit effort="76.94" velocity="1.571" /></joint>
-  <link name="elbow_flex_link">
-    <inertial>
-      <origin rpy="0 0 0" xyz="0.1279 0.0073 0.0000" />
-      <mass value="2.1299" />
-      <inertia ixx="0.0024" ixy="-0.0016" ixz="0.0" iyx="-0.0016" iyy="0.0082" iyz="-0.0" izx="0.0" izy="-0.0" izz="0.0084" />
-    </inertial>
-    <visual>
-      <origin rpy="0 0 0" xyz="0 0 0" />
-      <geometry>
-        <mesh filename="package://fetch_description/meshes/elbow_flex_link.dae" />
-      </geometry>
-      <material name="">
-        <color rgba="0.086 0.506 0.767 1" />
-      </material>
-    </visual>
-    <collision>
-      <origin rpy="0 0 0" xyz="0 0 0" />
-      <geometry>
-        <mesh filename="package://fetch_description/meshes/elbow_flex_link_collision.STL" />
-      </geometry>
-    </collision>
-  </link>
-  <joint name="elbow_flex_joint" type="revolute">
-    <origin rpy="0 0 0" xyz="0.133 0 0" />
-    <parent link="upperarm_roll_link" />
-    <child link="elbow_flex_link" />
-    <axis xyz="0 1 0" />
-  <limit effort="66.18" lower="-2.251" upper="2.251" velocity="1.521" /></joint>
-  <link name="forearm_roll_link">
-    <inertial>
-      <origin rpy="0 0 0" xyz="0.1097 -0.0266 0.0000" />
-      <mass value="1.6563" />
-      <inertia ixx="0.0016" ixy="-0.0003" ixz="0.0" iyx="-0.0003" iyy="0.003" iyz="-0.0" izx="0.0" izy="-0.0" izz="0.0035" />
-    </inertial>
-    <visual>
-      <origin rpy="0 0 0" xyz="0 0 0" />
-      <geometry>
-        <mesh filename="package://fetch_description/meshes/forearm_roll_link.dae" />
-      </geometry>
-      <material name="">
-        <color rgba="1 1 1 1" />
-      </material>
-    </visual>
-    <collision>
-      <origin rpy="0 0 0" xyz="0 0 0" />
-      <geometry>
-        <mesh filename="package://fetch_description/meshes/forearm_roll_link_collision.STL" />
-      </geometry>
-    </collision>
-  </link>
-  <joint name="forearm_roll_joint" type="continuous">
-    <origin rpy="0 0 0" xyz="0.197 0 0" />
-    <parent link="elbow_flex_link" />
-    <child link="forearm_roll_link" />
-    <axis xyz="1 0 0" />
-  <limit effort="29.35" velocity="1.571" /></joint>
-  <link name="wrist_flex_link">
-    <inertial>
-      <origin rpy="0 0 0" xyz="0.0882 0.0009 -0.0001" />
-      <mass value="1.725" />
-      <inertia ixx="0.0018" ixy="-0.0001" ixz="-0.0" iyx="-0.0001" iyy="0.0042" iyz="0.0" izx="-0.0" izy="0.0" izz="0.0042" />
-    </inertial>
-    <visual>
-      <origin rpy="0 0 0" xyz="0 0 0" />
-      <geometry>
-        <mesh filename="package://fetch_description/meshes/wrist_flex_link.dae" />
-      </geometry>
-      <material name="">
-        <color rgba="0.086 0.506 0.767 1" />
-      </material>
-    </visual>
-    <collision>
-      <origin rpy="0 0 0" xyz="0 0 0" />
-      <geometry>
-        <mesh filename="package://fetch_description/meshes/wrist_flex_link_collision.STL" />
-      </geometry>
-    </collision>
-  </link>
-  <joint name="wrist_flex_joint" type="revolute">
-    <origin rpy="0 0 0" xyz="0.1245 0 0" />
-    <parent link="forearm_roll_link" />
-    <child link="wrist_flex_link" />
-    <axis xyz="0 1 0" />
-  <limit effort="25.7" lower="-2.18" upper="2.18" velocity="2.268" /></joint>
-  <link name="wrist_roll_link">
-    <inertial>
-      <origin rpy="0 0 0" xyz="0.0095 0.0004 -0.0002" />
-      <mass value="0.1354" />
-      <inertia ixx="0.0001" ixy="0.0" ixz="0.0" iyx="0.0" iyy="0.0001" iyz="0.0" izx="0.0" izy="0.0" izz="0.0001" />
-    </inertial>
-    <visual>
-      <origin rpy="0 0 0" xyz="0 0 0" />
-      <geometry>
-        <mesh filename="package://fetch_description/meshes/wrist_roll_link.dae" />
-      </geometry>
-      <material name="">
-        <color rgba="1 1 1 1" />
-      </material>
-    </visual>
-    <collision>
-      <origin rpy="0 0 0" xyz="0 0 0" />
-      <geometry>
-        <mesh filename="package://fetch_description/meshes/wrist_roll_link_collision.STL" />
-      </geometry>
-    </collision>
-  </link>
-  <joint name="wrist_roll_joint" type="continuous">
-    <origin rpy="0 0 0" xyz="0.1385 0 0" />
-    <parent link="wrist_flex_link" />
-    <child link="wrist_roll_link" />
-    <axis xyz="1 0 0" />
-  <limit effort="7.36" velocity="2.268" /></joint>
-  <link name="gripper_link">
-    <inertial>
-      <origin rpy="0 0 0" xyz="-0.0900 -0.0001 -0.0017" />
-      <mass value="1.5175" />
-      <inertia ixx="0.0013" ixy="-0.0" ixz="0.0" iyx="-0.0" iyy="0.0019" iyz="-0.0" izx="0.0" izy="-0.0" izz="0.0024" />
-    </inertial>
-    <visual>
-      <origin rpy="0 0 0" xyz="0 0 0" />
-      <geometry>
-        <mesh filename="package://fetch_description/meshes/gripper_link.dae" />
-      </geometry>
-    </visual>
-    <collision>
-      <origin rpy="0 0 0" xyz="0 0 0" />
-      <geometry>
-        <mesh filename="package://fetch_description/meshes/gripper_link.STL" />
-      </geometry>
-    </collision>
-  </link>
-  <joint name="gripper_axis" type="fixed">
-    <origin rpy="0 0 0" xyz="0.16645 0 0" />
-    <parent link="wrist_roll_link" />
-    <child link="gripper_link" />
-    <axis xyz="0 1 0" />
-  </joint>
-  <link name="r_gripper_finger_link">
-    <inertial>
-      <origin rpy="0 0 0" xyz="-0.01 0 0" />
-      <mass value="0.0798" />
-      <inertia ixx="0.002" ixy="0" ixz="0" iyx="0.002" iyy="0" iyz="0" izx="0.002" izy="0" izz="0" />
-    </inertial>
-    <visual>
-      <origin rpy="0 0 0" xyz="0 0.101425 0" />
-      <geometry>
-        <mesh filename="package://fetch_description/meshes/r_gripper_finger_link.STL" />
-      </geometry>
-      <material name="">
-        <color rgba="0.356 0.361 0.376 1" />
-      </material>
-    </visual>
-    <collision>
-      <origin rpy="0 0 0" xyz="0 0.101425 0" />
-      <geometry>
-        <mesh filename="package://fetch_description/meshes/r_gripper_finger_link.STL" />
-      </geometry>
-    </collision>
-  </link>
-  <joint name="r_gripper_finger_joint" type="prismatic">
-    <origin rpy="0 0 0" xyz="0 0.015425 0" />
-    <parent link="gripper_link" />
-    <child link="r_gripper_finger_link" />
-    <axis xyz="0 1 0" />
-  <limit effort="60" lower="0.0" upper="0.05" velocity="0.05" /><dynamics damping="100.0" /></joint>
-  <link name="l_gripper_finger_link">
-    <inertial>
-      <origin rpy="0 0 0" xyz="-0.01 0 0" />
-      <mass value="0.0798" />
-      <inertia ixx="0.002" ixy="0" ixz="0" iyx="0.002" iyy="0" iyz="0" izx="0.002" izy="0" izz="0" />
-    </inertial>
-    <visual>
-      <origin rpy="0 0 0" xyz="0 -0.101425 0" />
-      <geometry>
-        <mesh filename="package://fetch_description/meshes/l_gripper_finger_link.STL" />
-      </geometry>
-      <material name="">
-        <color rgba="0.356 0.361 0.376 1" />
-      </material>
-    </visual>
-    <collision>
-      <origin rpy="0 0 0" xyz="0 -0.101425 0" />
-      <geometry>
-        <mesh filename="package://fetch_description/meshes/l_gripper_finger_link.STL" />
-      </geometry>
-    </collision>
-  </link>
-  <joint name="l_gripper_finger_joint" type="prismatic">
-    <origin rpy="0 0 0" xyz="0 -0.015425 0" />
-    <parent link="gripper_link" />
-    <child link="l_gripper_finger_link" />
-    <axis xyz="0 -1 0" />
-  <limit effort="60" lower="0.0" upper="0.05" velocity="0.05" /><dynamics damping="100.0" /></joint>
-  <link name="bellows_link">
-    <inertial>
-      <origin rpy="0 0 0" xyz="0.0191320000286228 -1.67219873481315E-16 -0.134861625443387" />
-      <mass value="0.169374038216602" />
-      <inertia ixx="0.00331159128762117" ixy="-8.9230964321455E-18" ixz="-5.38622201018293E-08" iyy="0.00174447292786627" iyz="-8.06964979976371E-17" izz="0.00169417568121457" />
-    </inertial>
-    <visual>
-      <origin rpy="0 0 0" xyz="0 0 0" />
-      <geometry>
-        <mesh filename="package://fetch_description/meshes/bellows_link.STL" />
-      </geometry>
-      <material name="">
-        <color rgba="0 0 0 1" />
-      </material>
-    </visual>
-    <collision>
-      <origin rpy="0 0 0" xyz="0 0 0" />
-      <geometry>
-        <mesh filename="package://fetch_description/meshes/bellows_link_collision.STL" />
-      </geometry>
-    </collision>
-  </link>
-  <joint name="bellows_joint" type="prismatic">
-    <origin rpy="0 0 0" xyz="0 0 0" />
-    <parent link="torso_lift_link" />
-    <child link="bellows_link" />
-    <axis xyz="0 0 -1" />
-  <limit effort="5.0" lower="0" upper="0.4" velocity="0.1" /></joint>
-  <link name="bellows_link2">
-    <inertial>
-      <origin rpy="0 0 0" xyz="0.0191320000286228 -1.67219873481315E-16 -0.134861625443387" />
-      <mass value="0.169374038216602" />
-      <inertia ixx="0.00331159128762117" ixy="-8.9230964321455E-18" ixz="-5.38622201018293E-08" iyy="0.00174447292786627" iyz="-8.06964979976371E-17" izz="0.00169417568121457" />
-    </inertial>
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