Commit message: Robotiq hand added

File: fetch_description/robots/fetch_robotiq_hands.urdf (robot description, URDF)
Before this commit: robot fetch_robotiq_hands, 63 links, 63 joints
Links:
- added link fake_robotiq_link
- link finger_1_link_0: geometry collision mesh filename=package://fetch_description/meshes/s-model_articulated/coll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; visual mesh filename=package://fetch_description/meshes/s-model_articulated/visu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
- link finger_1_link_1: geometry collision mesh filename=package://fetch_description/meshes/s-model_articulated/coll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; visual mesh filename=package://fetch_description/meshes/s-model_articulated/visu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
- link finger_1_link_2: geometry collision mesh filename=package://fetch_description/meshes/s-model_articulated/coll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; visual mesh filename=package://fetch_description/meshes/s-model_articulated/visu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
- link finger_1_link_3: geometry collision mesh filename=package://fetch_description/meshes/s-model_articulated/coll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; visual mesh filename=package://fetch_description/meshes/s-model_articulated/visu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
- link finger_2_link_0: geometry collision mesh filename=package://fetch_description/meshes/s-model_articulated/coll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; visual mesh filename=package://fetch_description/meshes/s-model_articulated/visu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
- link finger_2_link_1: geometry collision mesh filename=package://fetch_description/meshes/s-model_articulated/coll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; visual mesh filename=package://fetch_description/meshes/s-model_articulated/visu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
- link finger_2_link_2: geometry collision mesh filename=package://fetch_description/meshes/s-model_articulated/coll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; visual mesh filename=package://fetch_description/meshes/s-model_articulated/visu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
- link finger_2_link_3: geometry collision mesh filename=package://fetch_description/meshes/s-model_articulated/coll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; visual mesh filename=package://fetch_description/meshes/s-model_articulated/visu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
- link finger_middle_link_0: geometry collision mesh filename=package://fetch_description/meshes/s-model_articulated/coll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; visual mesh filename=package://fetch_description/meshes/s-model_articulated/visu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
- link finger_middle_link_1: geometry collision mesh filename=package://fetch_description/meshes/s-model_articulated/coll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; visual mesh filename=package://fetch_description/meshes/s-model_articulated/visu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
- link finger_middle_link_2: geometry collision mesh filename=package://fetch_description/meshes/s-model_articulated/coll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; visual mesh filename=package://fetch_description/meshes/s-model_articulated/visu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
- link finger_middle_link_3: geometry collision mesh filename=package://fetch_description/meshes/s-model_articulated/coll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; visual mesh filename=package://fetch_description/meshes/s-model_articulated/visu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
- link palm: geometry collision box size=0.1 0.1 0.1; visual mesh filename=package://fetch_description/meshes/s-model_articulated/visu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
Joints:
- joint gripper_axis: child palm -> fake_robotiq_link
- joint robotiq_hand_joint: origin xyz=-0.09 -0.0001 -0.0017 rpy=0 0 0 -> xyz=-0.09 -0.0001 -0.0017 rpy=-1.57079 0 0; parent wrist_roll_link -> fake_robotiq_link

File: fetch_description/robots/fetch_robotiq_hands.urdf.xacro (robot description, xacro)
@@ -3,7 +3,9 @@
   <xacro:include filename="$(find fetch_description)/robots/robotiq_hand.urdf.xacro"/>
   <xacro:freight_macro velocity_limit="17.4" />
-  <xacro:fetch gripper_link_name="palm"/>
-  <xacro:robotiq_hand prefix="" parent="wrist_roll_link" reflect="1">
-    <origin xyz="-0.09 -0.0001 -0.0017" rpy="0 0 0"/>
+  <xacro:fetch gripper_link_name="fake_robotiq_link"/>
+  <link name="fake_robotiq_link">
+  </link>
+  <xacro:robotiq_hand prefix="" parent="fake_robotiq_link" reflect="1">
+    <origin xyz="-0.09 -0.0001 -0.0017" rpy="-1.57079 0 0"/>
   </xacro:robotiq_hand>
 </robot>

File: fetch_description/robots/robotiq_hand.urdf.xacro (robot description, xacro)
@@ -14,5 +14,5 @@
         <origin xyz="0 0 0" rpy="0 0 0"/>
         <geometry>
-          <mesh filename="package://robotiq_hand_description/meshes/s-model_articulated/visual/link_0.STL" />
+          <mesh filename="package://fetch_description/meshes/s-model_articulated/visual/link_0.STL" />
         </geometry>
         <material name="green">
@@ -23,5 +23,5 @@
         <origin rpy="0 0 0" xyz="0 0 0"/>
         <geometry>
-          <mesh filename="package://robotiq_hand_description/meshes/s-model_articulated/collision/link_0.STL" />
+          <mesh filename="package://fetch_description/meshes/s-model_articulated/collision/link_0.STL" />
         </geometry>
         <material name="yellow">
@@ -44,5 +44,5 @@
         <origin rpy="0 0 ${3.1416/2}" xyz="0 0.05717 0"/>
         <geometry>
-          <mesh filename="package://robotiq_hand_description/meshes/s-model_articulated/visual/link_1.STL" />
+          <mesh filename="package://fetch_description/meshes/s-model_articulated/visual/link_1.STL" />
         </geometry>
         <material name="green"/>
@@ -51,5 +51,5 @@
         <origin rpy="0 0 ${3.1416/2}" xyz="0 0.05717 0"/>
         <geometry>
-          <mesh filename="package://robotiq_hand_description/meshes/s-model_articulated/collision/link_1.STL"/>
+          <mesh filename="package://fetch_description/meshes/s-model_articulated/collision/link_1.STL"/>
         </geometry>
         <material name="yellow">
@@ -78,5 +78,5 @@
         <origin rpy="0 0 ${3.1416/2}" xyz="0 0.03810 0.0075"/>
         <geometry>
-          <mesh filename="package://robotiq_hand_description/meshes/s-model_articulated/visual/link_2.STL" />
+          <mesh filename="package://fetch_description/meshes/s-model_articulated/visual/link_2.STL" />
         </geometry>
         <material name="green"/>
@@ -85,5 +85,5 @@
         <origin rpy="0 0 ${3.1416/2}" xyz="0 0.03810 0.0075"/>
           <geometry>
-            <mesh filename="package://robotiq_hand_description/meshes/s-model_articulated/collision/link_2.STL"/>
+            <mesh filename="package://fetch_description/meshes/s-model_articulated/collision/link_2.STL"/>
           </geometry>
         <material name="yellow"/>
@@ -110,5 +110,5 @@
         <origin xyz="0 0 0" rpy="0 0 0"/>
         <geometry>
-          <mesh filename="package://robotiq_hand_description/meshes/s-model_articulated/visual/link_3.STL" />
+          <mesh filename="package://fetch_description/meshes/s-model_articulated/visual/link_3.STL" />
         </geometry>
         <material name="green"/>
@@ -117,5 +117,5 @@
         <origin xyz="0 0 0" rpy="0 0 0"/>
         <geometry>
-          <mesh filename="package://robotiq_hand_description/meshes/s-model_articulated/collision/link_3.STL"/>
+          <mesh filename="package://fetch_description/meshes/s-model_articulated/collision/link_3.STL"/>
         </geometry>
         <material name="yellow"/>
@@ -555,5 +555,4 @@
           </dynamics>
           <xyz>0 0 1</xyz>
-          <use_parent_model_frame>false</use_parent_model_frame>
         </axis>
       </joint>
@@ -573,5 +572,4 @@
           </dynamics>
           <xyz>0 0 1</xyz>
-          <use_parent_model_frame>false</use_parent_model_frame>
         </axis>
       </joint>
@@ -591,5 +589,4 @@
           </dynamics>
           <xyz>0 0 1</xyz>
-          <use_parent_model_frame>false</use_parent_model_frame>
         </axis>
       </joint>
@@ -609,5 +606,4 @@
           </dynamics>
           <xyz>0 0 1</xyz>
-          <use_parent_model_frame>false</use_parent_model_frame>
         </axis>
       </joint>
@@ -627,5 +623,4 @@
           </dynamics>
           <xyz>0 0 1</xyz>
-          <use_parent_model_frame>false</use_parent_model_frame>
         </axis>
       </joint>
@@ -652,5 +647,5 @@
         <visual>
           <geometry>
-            <mesh filename="package://robotiq_hand_description/meshes/s-model_articulated/visual/palm.STL" />
+            <mesh filename="package://fetch_description/meshes/s-model_articulated/visual/palm.STL" />
           </geometry>
           <material name="green">
@@ -661,5 +656,5 @@
         <!-- <collision>
           <geometry>
-            <mesh filename="package://robotiq_hand_description/meshes/s-model_articulated/collision/palm.STL"/>
+            <mesh filename="package://fetch_description/meshes/s-model_articulated/collision/palm.STL"/>
           </geometry>
           <material name="yellow">
